Commit message: Gazebo OK 2020 jan26

File: rom1_description/urdf/rom1_description.urdf (robot description, URDF)
Before this commit: robot rom1, 5 links, 4 joints
Links:
- link base_link: mass 1.4621 -> 14.934
Joints:
- joint back_left_wheel_joint: origin xyz=-0.063652 0.22358 -0.027014 rpy=0 0 0 -> xyz=-0.05425 0.22 -0.029 rpy=0 0 0
- joint back_right_wheel_joint: origin xyz=-0.061796 -0.22142 -0.027014 rpy=0 0 0 -> xyz=-0.05425 -0.22 -0.028997 rpy=0 0 0
- joint front_left_wheel_joint: origin xyz=0.060348 0.22358 -0.027014 rpy=0 0 0 -> xyz=0.05425 0.22 -0.029 rpy=0 0 0
- joint front_right_wheel_joint: origin xyz=0.062204 -0.22142 -0.027014 rpy=0 0 0 -> xyz=0.05425 -0.22 -0.028997 rpy=0 0 0
